File: pacman/hardware/connectors.sch (KiCad schematic (older format))
At the start: 30 parts, among them J1 USB, J2 BACKPLANE CONNECTOR, J3 RJ12, P1 POWER, P2 CDETECT, P3 EXT I2C, P4 GPIO, P5 JTAG, P6 LDETECT, U14 TCA9617B

Commit message: Added in annotations about hardware changed
Other:
- note added: "Can be remove if using parallel connection\nwith the screen instead of I2C"
- note added: "Other GPIO pins\nthat are not used\nshould be broken\nout to this header"
Changed lines of the file:
@@
 Text Notes 4475 5550 0    100  ~ 0
 I2C PULLUP
+Text Notes 1750 6650 0    60   ~ 0
+Can be remove if using parallel connection\nwith the screen instead of I2C
+Text Notes 6400 4200 0    60   ~ 0
+Other GPIO pins\nthat are not used\nshould be broken\nout to this header
 $EndSCHEMATC
