File: pacman/hardware/pacman-main.sch (KiCad schematic (older format))
At the start: 21 parts, among them SW1 RESET, U1 AT90CAN128-M, U2 ADM6320, X1 10MHz

Commit message: Added in annotations about hardware changed
Other:
- note added: "These IOs can be brought\nout to control a screen\ninstead of using an I2C\nexpander attached to\nthe screen"
Changed lines of the file:
@@
 Text Label 3325 7675 2    60   ~ 0
 PB4
+Text Notes 7150 4100 0    60   ~ 0
+These IOs can be brought\nout to control a screen\ninstead of using an I2C\nexpander attached to\nthe screen
 $EndSCHEMATC
